File: PCB/tester/DUT.kicad_sch (KiCad schematic)
At the start: 72 parts, among them J3 6pin_hd, J4 Conn_02x03_Odd_Even, J5 MotorCkeck1, J6 MotorCkeck2, J7 Conn_01x02_Socket, K1 Relay SPDT, K2 Relay SPDT, K3 Relay SPDT, Q2 PMF170XP,115, Q3 DMN63D8L-7, Q4 DMN63D8L-7, Q5 DMN63D8L-7, Q6 DMN63D8L-7, U6 THS4281, U7 THS4281, U8 THS4281, U9 ZXCT1082

Commit message: Final details and production files
Co-Authored-By: David Palma <78764277+davidpalma666@users.noreply.github.com>
Parts:
- J4: value Conn_02x03_Odd_Even -> 61300621021
- J5: value MotorCkeck1 -> PPTC051LFBN-RC
- J6: value MotorCkeck2 -> 61300511021
- J7: value Conn_01x02_Socket -> PPTC021LFBN-RC
- R24, R25, R32: MPN ERJ-2RKF5101X -> RT0402BRD075K1L; OEPSPN OEPS020173 -> OEPS020203; Tolerance 1% -> 0.1%
- R45, R49: Tolerance 0.1% -> 1%
- R47: value 4k3 -> 4.3k; Tolerance 1% -> 5%
