File: PCB/tester/DUT.kicad_sch (KiCad schematic)
At the start: 72 parts, among them J3 6pin_hd, J4 61300621021, J5 PPTC051LFBN-RC, J6 61300511021, J7 PPTC021LFBN-RC, K1 Relay SPDT, K2 Relay SPDT, K3 Relay SPDT, Q2 PMF170XP,115, Q3 DMN63D8L-7, Q4 DMN63D8L-7, Q5 DMN63D8L-7, Q6 DMN63D8L-7, U6 THS4281, U7 THS4281, U8 THS4281, U9 ZXCT1082

Commit message: Update 1N4148 part numbers
Replace obsolete 1N4148 :
OEPS030017 -> OEPS030052
1N4148WX-TP -> 1N4148WS-E3-18
Parts:
- D10, D11, D9: MPN 1N4148WX-TP -> 1N4148WS-E3-18; OEPSPN OEPS030017 -> OEPS030052
Changed lines of the file:
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@@
 			)
 		)
-		(property "OEPSPN" "OEPS030017"
+		(property "OEPSPN" "OEPS030052"
 			(at 71.12 162.56 90)
 			(hide yes)
@@
 			)
 		)
-		(property "MPN" "1N4148WX-TP"
+		(property "MPN" "1N4148WS-E3-18"
 			(at 71.12 162.56 90)
 			(hide yes)
@@
 			)
 		)
-		(property "OEPSPN" "OEPS030017"
+		(property "OEPSPN" "OEPS030052"
 			(at 49.53 129.54 90)
 			(hide yes)
@@
 			)
 		)
-		(property "MPN" "1N4148WX-TP"
+		(property "MPN" "1N4148WS-E3-18"
 			(at 49.53 129.54 90)
 			(hide yes)
@@
 			)
 		)
-		(property "OEPSPN" "OEPS030017"
+		(property "OEPSPN" "OEPS030052"
 			(at 189.23 132.08 90)
 			(hide yes)
@@
 			)
 		)
-		(property "MPN" "1N4148WX-TP"
+		(property "MPN" "1N4148WS-E3-18"
 			(at 189.23 132.08 90)
 			(hide yes)
