File: PCB/tester/FED3 tester.kicad_sch (KiCad schematic)
At the start: 31 parts, among them J1 USB4105-GF-A, U1 FT232RL, U2 LP5907MFX-3.3, U3 LP5907MFX-3.3, U4 TPS73801DCQR

Commit message: Final details and production files
Co-Authored-By: David Palma <78764277+davidpalma666@users.noreply.github.com>
Parts:
- C14: TempCo X5R -> X7R
- L1, L2: value 40R@100MHz -> MI0805K400R-10
- R1, R3: MPN ERJ-2RKF5101X -> RT0402BRD075K1L; OEPSPN OEPS020173 -> OEPS020203; Tolerance 1% -> 0.1%
- R7: value 8k2 -> 8.2k
- U1: value FT232RL -> FT232RNL-REEL
Other:
- moved on the sheet: C3, R2
