File: PCB/tester/main core.kicad_sch (KiCad schematic)
At the start: 44 parts, among them J2 Conn_02x03_Odd_Even, Q1 DMN63D8L-7, SW1 SW_SPST, SW2 SW_SPST, SW3 SW_SPST, SW4 SW_SPST, SW5 SW_SPST, SW6 SW_SPST, SW7 SW_SPST, SW8 SW_SPST, SW9 SW_SPST, U5 ATXMEGA32A4U-MH

Commit message: Final details and production files
Co-Authored-By: David Palma <78764277+davidpalma666@users.noreply.github.com>
Parts:
- D8: MPN VFHR1116P-4C82A-TR -> 5990010007F; OEPSPN OEPS030038 -> OEPS030044
- J2: value Conn_02x03_Odd_Even -> PR20203VBDN
- R10, R11, R12, R16, R9: value 2k -> 330R; MPN ERJ-2RKF2001X -> CRCW0402330RFKEDHP; OEPSPN OEPS020007 -> OEPS020191
- R17: value 10k -> 560R; MPN CPF0402B10KE1 -> CRCW0402560RFKED; OEPSPN OEPS020043 -> OEPS020193; Tolerance 0.1% -> 1%
- SW1, SW2, SW3, SW4, SW5, SW6, SW7, SW8, SW9: value SW_SPST -> TL3305BF260QG
