File: PCB/tester/FED3 tester.kicad_pcb (KiCad board)
At the start: 4 copper layers, 108 x 134.4 mm, 166 parts, among them J1 USB4105-GF-A, J2 Conn_02x03_Odd_Even, J3 6pin_hd, J4 Conn_02x03_Odd_Even, J5 MotorCkeck1, J6 MotorCkeck2, J7 Conn_01x02_Socket, K1 Relay SPDT, K2 Relay SPDT, K3 Relay SPDT, Q1 DMN63D8L-7, Q2 PMF170XP,115, Q3 DMN63D8L-7, Q4 DMN63D8L-7, Q5 DMN63D8L-7, Q6 DMN63D8L-7, SW1 SW_SPST, SW2 SW_SPST, SW3 SW_SPST, SW4 SW_SPST, SW5 SW_SPST, SW6 SW_SPST, SW7 SW_SPST, SW8 SW_SPST, SW9 SW_SPST, U1 FT232RL, U2 LP5907MFX-3.3, U3 LP5907MFX-3.3, U4 TPS73801DCQR, U5 ATXMEGA32A4U-MH, U6 THS4281, U7 THS4281, U8 THS4281, U9 ZXCT1082

Commit message: Final details and production files
Co-Authored-By: David Palma <78764277+davidpalma666@users.noreply.github.com>
Parts:
- J2: value Conn_02x03_Odd_Even -> PR20203VBDN
- J4: value Conn_02x03_Odd_Even -> 61300621021
- J5: value MotorCkeck1 -> PPTC051LFBN-RC
- J6: value MotorCkeck2 -> 61300511021
- J7: value Conn_01x02_Socket -> PPTC021LFBN-RC
- L1, L2: value 40R@100MHz -> MI0805K400R-10
- R10, R11, R12, R16, R9: value 2k -> 330R
- R17: value 10k -> 560R
- R47: value 4k3 -> 4.3k
- R7: value 8k2 -> 8.2k
- SW1, SW2, SW3, SW4, SW5, SW6, SW7, SW8, SW9: value SW_SPST -> TL3305BF260QG
- U1: value FT232RL -> FT232RNL-REEL
- moved C28 91.2 mm to (130.5, 41.9), turned to 90 degrees
- moved C27 82.1 mm to (131.2, 49.2), turned to 0 degrees
- moved C23 62.3 mm to (128.9, 53.7)
- moved C20 61.2 mm to (126.3, 58.9)
- moved C22 57.8 mm to (127.6, 54.8)
- moved C21 54.3 mm to (127.8, 58.9)
- moved C26 46.7 mm to (131.1, 50.8), turned to 0 degrees
- moved C25 42.1 mm to (129.6, 51.9), turned to 0 degrees
- moved C16 36.8 mm to (124.6, 58.9)
- moved OSC1 0.27 mm to (125.5, 41.6)
- moved C24 0.15 mm to (128.4, 42.0)
Routing:
- net /main core/Prog_OK: track 99.1 -> 89.9 mm
- net GND: track 220.7 -> 214.3 mm, vias 237 -> 242
- net /main core/RGBW_NOK: track 96.2 -> 90.9 mm
- net /main core/Buzzer_OK: track 94.4 -> 98.5 mm
- net /main core/Buzzer_NOK: track 127.0 -> 123.6 mm, vias 3 -> 4
- net /main core/RGBW_OK: track 71.3 -> 72.6 mm
- net /main core/Prog_NOK: track 78.3 -> 79.5 mm
- net /main core/Motor_OK: track 54.7 -> 55.5 mm
- added copper zone on F.Cu, net GND

Commit message: Replace R13 100R with 1R and update BOM/metadata
Parts:
- R13: value 100R -> 1R
Changed lines of the file:
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@@
 			)
 		)
-		(property "Value" "100R"
+		(property "Value" "1R"
 			(at 0 1.17 90)
 			(unlocked yes)
@@
 			)
 		)
-		(property "Description" "RESISTOR:   SMD 0402 100Ω ±1% 0.250W   [RCS0402100RFKED] [SMD]"
+		(property "Description" "RESISTOR:   SMD 0402 1Ω ±1% 0.200W   [CRCW04021R00FKEDHP] [SMD]"
 			(at 0 0 90)
 			(unlocked yes)
@@
 			)
 		)
-		(property "MPN" "RCS0402100RFKED"
+		(property "MPN" "CRCW04021R00FKEDHP"
 			(at 0 0 90)
 			(unlocked yes)
@@
 			)
 		)
-		(property "OEPSPN" "OEPS020028"
+		(property "OEPSPN" "OEPS020224"
 			(at 0 0 90)
 			(unlocked yes)
